File: energy_meter/energy_meter.kicad_sch (KiCad schematic)
At the start: 19 parts

Commit message: Schematic progress
Parts:
- added C10, C4, C8, C9: 0.022u, symbol Device:C
- added C11, C12, C13: C, symbol Device:C
- added C14, C16, C18, C20: 0.1u, symbol Device:C
- added C15, C17, C19, C21: 4.7u, symbol Device:C
- added C5: 51p, symbol Device:C
- added CR3, CR4: MMBD4148SE, SOT-23TO-236_318-AT_OSI, symbol MMBD4148SE:MMBD4148SE
- added D1, D2, D3, D4, D5: LED, symbol Device:LED
- added FB2: FerriteBead, symbol Device:FerriteBead
- added R10, R12, R14, R9: 200k, symbol Device:R_US
- added R15, R16, R19, R20: 1k, symbol Device:R_US
- added R17, R18: 40.2, symbol Device:R_US
- added R21: 10K, symbol Device:R_US
- added R22, R23: R_US, symbol Device:R_US
- added R24, R25, R26: 3K, symbol Device:R_US
- added R27, R28: 3V, symbol Device:R_US
- added U1: ADE9000ACPZ, ADE9000ACPZ_ADI, symbol ADE9000:ADE9000ACPZ
- added Y1: Crystal_GND24, symbol Device:Crystal_GND24
Connections:
- net GND: now also C10.1, C11.2, C12.2, C13.2, C14.2, C15.2, C16.2, C17.2, C18.2, C19.2, C20.2, C21.2, C4.2, C8.2, C9.2, CR3.3, CR4.3, D3.1 (K), D4.1 (K), R15.1, R16.1, R17.2, R18.1, R21.2, U1.15 (REFGND), U1.2 (DGND), U1.26 (AGND), U1.28 (GND), U1.41 (EPAD), Y1.2, Y1.4
- net IAN: now also U1.8 (IAN)
- net IAP: now also U1.7 (IAP)
- net VAN: now also U1.19 (VAN)
- net VAP: now also U1.20 (VAP)
- new net: CR3.1, CR4.2, R17.1, R19.1
- new net: CR3.2, CR4.1, R18.2, R20.1
- new net: C12.1, U1.30 (CLKOUT), Y1.1
- new net: C13.1, U1.29 (CLKIN), Y1.3
- new net: R10.2, R12.1
- new net: R12.2, R14.1
- new net: D2.2 (A), R25.2
- new net: FB2.1, R9.1
- new net: R10.1, R9.2
- new net: D1.2 (A), R24.2
- new net: D3.2 (A), R26.2
- new net: D5.2 (A), R28.2
- new net: D4.2 (A), R27.2
- new net: R23.1, U1.40 (*SS)
- new net +3V3_ADE: R22.1, R23.2, R24.1, R25.1, R28.1, U1.27 (VDD), U1.4 (PM0)
- new net +3V3_ISO: C20.1, C21.1
- new net 3V3_ISO: U1.1 (PULL_HIGH)
- new net AVDDOUT: C16.1, C17.1, U1.25 (AVDDOUT)
- new net CF1_ADE: U1.33 (CF1)
- new net CF2_ADE: U1.34 (CF2)
- new net DREADY_ADE: R27.1, U1.36 (CF4/*EVENT/DREADY)
- new net DVDDOUT: C14.1, C15.1, U1.3 (DVDDOUT)
- new net IBN: C10.2, R20.2, U1.10 (IBN)
- new net IBP: C9.1, R19.2, U1.9 (IBP)
- new net IQR1_ADE: D2.1 (K)
- new net IRQ0_ADE: D1.1 (K), D5.1 (K), U1.31 (*IRQ0)
- new net IRQ1_ADE: U1.32 (*IRQ1)
- new net MISO_ADE: U1.38 (MISO)
- new net MOSI_ADE: U1.39 (MOSI)
- new net PM1_ADE: R21.1, U1.5 (PM1)
- new net REF: C18.1, C19.1, U1.16 (REF)
- new net RESET_ADE: C11.1, R22.2, U1.6 (*RESET)
- new net SCLK_ADE: U1.37 (SCLK)
- new net VBN: C5.2, C8.1, R16.2, U1.21 (VBN)
- new net VBP: C4.1, C5.1, R14.2, R15.2, U1.22 (VBP)
- new net ZX_ADE: R26.1, U1.35 (CF3/ZX)
- no-connect marks 0 -> 6
Other:
- added sheet energy_meter2 (energy_meter2.kicad_sch)

Commit message: Progress in schematic
Parts:
- added C22, C23, C24, C26, C28, C30, C31, C33, C35: 0.1u, Capacitor_SMD:C_0805_2012Metric_Pad1.18x1.45mm_HandSolder, symbol Device:C
- added C25, C27, C29, C32, C34: 10u, Capacitor_SMD:C_0805_2012Metric_Pad1.18x1.45mm_HandSolder, symbol Device:C
- added H1, H2, H3, H4: MountingHole, MountingHole:MountingHole_3.2mm_M3, symbol Mechanical:MountingHole
- added IC1: ADUM4151BRIZ, ADUM4151BRIZ:SOIC127P1031X264-20N, symbol ADUM4151BRIZ:ADUM4151BRIZ
- added IC2: ADUM6404ARIZ, ADUM6404ARIZ:SOIC127P1032X265-16N, symbol ADUM6404ARIZ:ADUM6404ARIZ
- added IC3: ADP122AUJZ-3.3-R7, ADP122AUJZ-3.3-R7:SOT95P280X100-5N, symbol ADP122AUJZ-3.3-R7:ADP122AUJZ-3.3-R7
- added J1, J2: Screw_Terminal_01x02, TerminalBlock_Phoenix:TerminalBlock_Phoenix_MKDS-1,5-2_1x02_P5.00mm_Horizontal, symbol Connector:Screw_Terminal_01x02
- added R29: 10k, Resistor_SMD:R_0805_2012Metric_Pad1.20x1.40mm_HandSolder, symbol Device:R_US
- added T1, T2: T60404-E4626-X502, T60404E4626X502:T60404E4626X502, symbol Current Transformer:T60404-E4626-X502
- added TP1, TP10, TP11, TP12, TP13, TP14, TP15, TP16, TP17, TP18, TP19, TP2, TP20, TP21, TP22, TP23, TP24, TP25, TP26, TP27, TP28, TP29, TP3, TP30, TP31, TP32, TP4, TP5, TP6, TP7, TP8, TP9: TestPoint, TestPoint:TestPoint_Pad_D1.5mm, symbol Connector:TestPoint
- added U2, U3: SN74LV4T125PWR, SN74LV4T125PWR:PW0014A_N, symbol SN74LV4T125PWR:SN74LV4T125PWR
- C1, C10, C14, C15, C16, C17, C18, C19, C2, C20, C21, C3, C4, C5, C6, C7, C8, C9: footprint (none) -> Capacitor_SMD:C_0805_2012Metric_Pad1.18x1.45mm_HandSolder
- C11: value C -> 1u; footprint (none) -> Capacitor_SMD:C_0805_2012Metric_Pad1.18x1.45mm_HandSolder
- C12, C13: value C -> 18p; footprint (none) -> Capacitor_SMD:C_0805_2012Metric_Pad1.18x1.45mm_HandSolder
- CR1, CR2, CR3, CR4: footprint SOT-23TO-236_318-AT_OSI -> MMBD4148SE:SOT-23TO-236_318-AT_OSI
- D1, D2, D3, D4, D5: footprint (none) -> LED_SMD:LED_0603_1608Metric_Pad1.05x0.95mm_HandSolder
- FB1, FB2, FB3: footprint (none) -> Inductor_SMD:L_0805_2012Metric_Pad1.05x1.20mm_HandSolder
- R1, R10, R12, R14, R2, R3, R4, R9: footprint (none) -> Resistor_SMD:R_2010_5025Metric_Pad1.40x2.65mm_HandSolder
- R11, R13, R15, R16, R17, R18, R19, R20, R21, R5, R6, R7, R8: footprint (none) -> Resistor_SMD:R_0805_2012Metric_Pad1.20x1.40mm_HandSolder
- R22, R23: value R_US -> 10k; footprint (none) -> Resistor_SMD:R_0805_2012Metric_Pad1.20x1.40mm_HandSolder
- R24, R25, R26: footprint (none) -> Resistor_SMD:R_0603_1608Metric_Pad0.98x0.95mm_HandSolder
- R27, R28: value 3V -> 3k; footprint (none) -> Resistor_SMD:R_0603_1608Metric_Pad0.98x0.95mm_HandSolder
- U1: footprint ADE9000ACPZ_ADI -> ade9000:ADE9000ACPZ_ADI-M
- Y1: footprint (none) -> Crystal:Crystal_SMD_3225-4Pin_3.2x2.5mm_HandSoldering
Connections:
- net 3V3_ISO is gone; now on net +3V3_ISO: U1.1 (PULL_HIGH)
- net +3V3_ADE: now also C22.1, C34.1, C35.1, IC1.20 (VDD2), IC2.10 (VSEL), IC3.5 (VOUT)
- net +3V3_ISO: now also C23.2, C31.1, IC1.1 (VDD1), U3.14 (VCC)
- net DREADY_ADE: now also TP10.1, U2.5 (2A)
- net GND: now also C22.2, C24.2, C25.2, C26.2, C27.2, C32.2, C33.2, C34.2, C35.2, IC1.11 (GND2_1), IC1.12 (VIC), IC1.19 (GND2_2), IC2.15 (GNDISO_2), IC2.9 (GNDISO_1), IC3.2 (GND), TP15.1, TP16.1, U2.1 (1OE_N), U2.10 (3OE_N), U2.13 (4OE_N), U2.4 (2OE_N), U2.7 (GND)
- net IRQ0_ADE: now also TP12.1, U2.9 (3A)
- net IRQ1_ADE: now also TP11.1, U2.12 (4A)
- net MISO_ADE: now also IC1.16 (SO), TP5.1, TP6.1
- net MOSI_ADE: now also IC1.17 (SI), TP3.1, TP4.1
- net PM1_ADE: now also IC1.14 (VOA), TP13.1
- net RESET_ADE: now also IC1.13 (VOB), TP9.1
- net SCLK_ADE: now also IC1.18 (SCLK), TP1.1, TP2.1
- net ZX_ADE: now also TP14.1, U2.2 (1A)
- net at CR1.2, CR2.1, R13.1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: now also T1.4
- net at CR1.1, CR2.2, R11.1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: now also T1.1
- net at CR3.1, CR4.2, R17.1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: now also T2.1
- net at CR3.2, CR4.1, R18.2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: now also T2.4
- net VB: now reaches FB2.2
- net VB: now also J1.2 (Pin_2)
- net SS_ADE: now reaches R23.1, U1.40 (*SS)
- net SS_ADE: now also IC1.15 (~{SSS}), TP7.1, TP8.1
- net VA: now reaches FB1.2
- net VA: now also J1.1 (Pin_1)
- net EARTH: now reaches FB3.2
- net EARTH: now also J2.1 (Pin_1), J2.2 (Pin_2)
- new net: IC2.6 (VOD), U3.12 (4A)
- new net: IC2.3 (VOA), U3.2 (1A)
- new net: IC2.4 (VOB), U3.5 (2A)
- new net: IC2.5 (VOC), U3.9 (3A)
- new net: IC2.11 (VID), U2.6 (2Y)
- new net: IC2.12 (VIC), U2.3 (1Y)
- new net: IC2.13 (VIB), U2.11 (4Y)
- new net: IC2.14 (VIA), U2.8 (3Y)
- new net: C30.2, IC2.7 (VDDL)
- new net +5V_ADE: C24.1, C25.1, C26.1, C27.1, C32.1, C33.1, IC2.16 (VISO), IC3.1 (VIN), IC3.3 (EN), U2.14 (VCC)
- new net +5V_PICO: C28.1, C29.1, IC2.1 (VDD1)
- new net DREADY_ISO: TP28.1, U3.11 (4Y)
- new net GNDA: C23.1, C28.2, C29.2, C30.1, C31.2, IC1.10 (GND1_2), IC1.2 (GND1_1), IC2.2 (GND1_1), IC2.8 (GND1_2), R29.1, TP31.1, TP32.1, U3.1 (1OE_N), U3.10 (3OE_N), U3.13 (4OE_N), U3.4 (2OE_N), U3.7 (GND)
- new net IRQ0_ISO: TP30.1, U3.3 (1Y)
- new net IRQ1_ISO: TP29.1, U3.6 (2Y)
- new net MISO_ISO: IC1.5 (MI), TP21.1, TP22.1
- new net MOSI_ISO: IC1.4 (MO), TP19.1, TP20.1
- new net PM1_ISO: IC1.7 (VIA), R29.2, TP26.1
- new net RESET_ISO: IC1.8 (VIB), TP25.1
- new net SCLK_ISO: IC1.3 (MCLK), TP17.1, TP18.1
- new net SS_ISO: IC1.6 (~{MSS}), TP23.1, TP24.1
- new net ZX_ISO: TP27.1, U3.8 (3Y)
- no-connect marks 6 -> 11
Other:
- removed sheet energy_meter2
- note added: "3V3 <- 5V <----- 5V <- 3V3 Why?"
- note added: "3V3 from ADE9000, converted to 5V and sent to isopower"
- note added: "3V3 signals"
- note added: "5V from isopower, converted to 3V3 and sent to Pico"
- note added: "ADE9000 and LED peripherals"
- note added: "ADE9000 will always enter Power Mode 0 (PM1, PM0 = 01) unless PM1 is set. PM0 is normal operation"
- note added: "Current Channels"
- note added: "HOT/LIVE SIDE"
- note added: "Is this even needed if we don't need the level shift"
- note added: "Level shifter and isolator"
- note added: "SAFE/MCU SIDE"
- note added: "SPI isolator"
- note added: "Voltage Channels"
- note added: "What should this connector be?"
- moved on the sheet: C1, C10, C11, C12, C13, C14, C15, C16, C17, C18, C19, C2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

Commit message: Finish up schematic
Parts:
- added C36: 1u, Capacitor_SMD:C_0805_2012Metric_Pad1.18x1.45mm_HandSolder, symbol Device:C
- added C37: 4.7u, Capacitor_SMD:C_0805_2012Metric_Pad1.18x1.45mm_HandSolder, symbol Device:C
- added C38, C39, C41, C44: 0.1u, Capacitor_SMD:C_0805_2012Metric_Pad1.18x1.45mm_HandSolder, symbol Device:C
- added C40, C42: 10u, Capacitor_SMD:C_0805_2012Metric_Pad1.18x1.45mm_HandSolder, symbol Device:C
- added C43: 22u, Capacitor_SMD:C_0805_2012Metric_Pad1.18x1.45mm_HandSolder, symbol Device:C
- added D6, D7, D8: D_Schottky, Diode_SMD:D_SOD-323_HandSoldering, symbol Device:D_Schottky
- added IC4: 24LC32A_SN, 24LC32A_SN:SOIC127P600X175-8N, symbol 24LC32A_SN:24LC32A_SN
- added J3: ZX62-AB-5PA_31_, microUSB:ZX62AB5PA31, symbol microUSB:ZX62-AB-5PA_31_
- added R30, R31, R32, R33: 10k, Resistor_SMD:R_0805_2012Metric_Pad1.20x1.40mm_HandSolder, symbol Device:R_US
- added SW1: SW_Push, Button_Switch_THT:SW_PUSH_6mm, symbol Switch:SW_Push
- added U4: Pico_SMD_NODEBUG, RPi Pico:RPi_PicoW_SMD, symbol RPi Pico:Pico_SMD_NODEBUG
Connections:
- net +3V3_ISO: now also C36.1, C37.1, C38.1, C39.1, C40.1, D8.2 (A), IC4.8 (VCC), R30.1, R31.1, R32.1, R33.1
- net +5V_PICO: now also C41.1, C42.1, C43.1, C44.1, J3.1
- net DREADY_ISO: now also U4.17 (GPIO13)
- net GNDA: now also C37.2, C38.2, C39.2, C40.2, C41.2, C42.2, C43.2, C44.2, IC4.1 (A0), IC4.2 (A1), IC4.3 (A2), IC4.4 (VSS), IC4.7 (WP), J3.5, J3.MP1, J3.MP2, J3.MP3, J3.MP4, J3.MP5, J3.MP6, SW1.1, U4.13 (GND), U4.18 (GND), U4.23 (GND), U4.28 (GND), U4.3 (GND), U4.33 (AGND), U4.38 (GND), U4.8 (GND)
- net IRQ0_ISO: now also U4.14 (GPIO10)
- net IRQ1_ISO: now also U4.15 (GPIO11)
- net MISO_ISO: now also U4.11 (GPIO8)
- net MOSI_ISO: now also U4.10 (GPIO7)
- net PM1_ISO: now also U4.19 (GPIO14)
- net RESET_ISO: now also C36.2, D6.2 (A), D7.2 (A), R30.2
- net SCLK_ISO: now also U4.9 (GPIO6)
- net SS_ISO: now also R33.2, U4.12 (GPIO9)
- net ZX_ISO: now also U4.16 (GPIO12)
- new net: D8.1 (K), U4.39 (VSYS)
- new net: D6.1 (K), SW1.2
- new net RESET_PICO: D7.1 (K), U4.30 (RUN)
- new net SCL_PICO: IC4.6 (SCL), R32.2, U4.7 (GPIO5)
- new net SDA_PICO: IC4.5 (SDA), R31.2, U4.6 (GPIO4)
Other:
- note added: "Do we need this with RPi Pico having 2MB flash?"

Commit message: Add lipo battery terminal
Parts:
- added C45, C47: 10u, Capacitor_SMD:C_0805_2012Metric_Pad1.18x1.45mm_HandSolder, symbol Device:C
- added C46, C48: 0.1u, Capacitor_SMD:C_0805_2012Metric_Pad1.18x1.45mm_HandSolder, symbol Device:C
- added IC5: ADP122AUJZ-3.3-R7, ADP122AUJZ-3.3-R7:SOT95P280X100-5N, symbol ADP122AUJZ-3.3-R7:ADP122AUJZ-3.3-R7
- added J4: XT30, Connector_AMASS:AMASS_XT30PW-M_1x02_P2.50mm_Horizontal, symbol Connector_Generic:Conn_01x02
- J3: value ZX62-AB-5PA_31_ -> MicroUSB
Connections:
- net +5V_PICO is gone; now on net GNDA: C28.1, C29.1, C41.1, C42.1, C43.1, C44.1, IC2.1 (VDD1), J3.1
- net +3V3_ADE: no longer IC2.10 (VSEL)
- net +3V3_ISO: now also C47.1, C48.1, IC5.5 (VOUT)
- net +5V_ADE: now also IC2.10 (VSEL)
- net GND: now also C45.2, C46.2, C47.2, C48.2, IC5.2 (GND)
- net GNDA: now also J4.1 (Pin_1)
- new net V_BATT: C45.1, C46.1, IC5.1 (VIN), IC5.3 (EN), J4.2 (Pin_2)
Other:
- note added: "If we do not need to generate 5V, we can use 3.7V(4.2V) input from LiPo 1S battery to power the MCU and ADE9000"

Commit message: Minor changes
Connections:
- net DREADY_ADE: now also U2.12 (4A); no longer U2.5 (2A)
- net GND: now also D5.1 (K)
- net IRQ0_ADE: now also U2.2 (1A); no longer D5.1 (K), U2.9 (3A)
- net IRQ1_ADE: now also U2.5 (2A); no longer U2.12 (4A)
- net ZX_ADE: now also U2.9 (3A); no longer U2.2 (1A)
- net at IC2.11 (VID): now also U2.11 (4Y); no longer U2.6 (2Y)
- net at IC2.12 (VIC): now also U2.8 (3Y); no longer U2.3 (1Y)
- net at IC2.13 (VIB): now also U2.6 (2Y); no longer U2.11 (4Y)
- net at IC2.14 (VIA): now also U2.3 (1Y); no longer U2.8 (3Y)
Other:
- note added: "--------->"
- note added: "<------- Logic flow"
- note added: "ADE9000 and peripherals"
- note added: "For 3.3V output at VISO, this pin needs to be at GND"
- note added: "If we provide just 3.3V here, the buffer will produce outputs at 3.3V logic. This can then be fed to the isolator"
- note added: "Level shifter"
- note added: "Power flow ------->"
- note added: "Power isolator"
- note added: "This device can operate at either 3.3V or 5V supply. It can either do 5 -> 5 or 5 -> 3.3 or 3.3 -> 3.3"
- note removed: "ADE9000 and LED peripherals"
- note removed: "Level shifter and isolator"
- moved on the sheet: C26, C27, C43, C44, J3, U2

Commit message: Minor changes
Parts:
- added J5: VA, Connector:Banana_Cliff_FCR7350R_S16N-PC_Horizontal, symbol Connector_Generic_MountingPin:Conn_01x01_MountingPin
- added J6: VB, Connector:Banana_Cliff_FCR7350R_S16N-PC_Horizontal, symbol Connector_Generic_MountingPin:Conn_01x01_MountingPin
- added J7: EARTH, Connector:Banana_Cliff_FCR7350B_S16N-PC_Horizontal, symbol Connector_Generic_MountingPin:Conn_01x01_MountingPin
Connections:
- net EARTH: now also J7.1 (Pin_1)
- net GNDA: no longer C28.1, C29.1, C41.1, C42.1, C43.1, C44.1, IC2.1 (VDD1), J3.1
- net VA: now also J5.1 (Pin_1)
- net VB: now also J6.1 (Pin_1)
- net +5V_PICO: now reaches C30.2, IC2.7 (VDDL)
- net +5V_PICO: now also C28.1, C29.1, C41.1, C42.1, C43.1, C44.1, IC2.1 (VDD1), J3.1
- no-connect marks 11 -> 14
Other:
- added sheet central_unit (central_unit.kicad_sch)
- note added: "What? Why is 3V3_ISO here?"
- moved on the sheet: J1, J2

Commit message: Minor changes
Parts:
- added J8: 5V_SMPS, symbol Connector:Screw_Terminal_01x02
Connections:
- net +3V3_ISO: no longer D8.2 (A)
- net +5V_PICO: now also D8.2 (A), J8.2 (Pin_2)
- net GNDA: now also J8.1 (Pin_1)
Other:
- note added: "----->"
- note removed: "--------->"
Changed lines of the file:
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@@
     (stroke (width 0) (type default))
   )
+  (wire (pts (xy 259.08 228.6) (xy 259.08 229.87))
+    (stroke (width 0) (type default))
+  )
   (wire (pts (xy 490.22 304.8) (xy 491.49 304.8))
     (stroke (width 0) (type default))
@@
     (stroke (width 0) (type default))
   )
+  (wire (pts (xy 256.54 226.06) (xy 259.08 226.06))
+    (stroke (width 0) (type default))
+  )
   (wire (pts (xy 238.76 226.06) (xy 238.76 228.6))
     (stroke (width 0) (type default))
@@
     (stroke (width 0) (type default))
   )
+  (wire (pts (xy 256.54 228.6) (xy 259.08 228.6))
+    (stroke (width 0) (type default))
+  )
   (wire (pts (xy 322.58 96.52) (xy 361.95 96.52))
     (stroke (width 0) (type default))
@@
     (effects (font (size 1.27 1.27)) (justify left bottom))
   )
-  (text "--------->" (at 250.19 215.9 90)
+  (text "----->" (at 250.19 208.28 90)
     (effects (font (size 1.27 1.27)) (justify left bottom))
   )
@@
   )
   (text "If we do not need to generate 5V,\nwe can use 3.7V(4.2V) input from\nLiPo 1S battery to power the MCU\nand ADE9000\n"
-    (at 242.57 223.52 0)
+    (at 242.57 215.9 0)
     (effects (font (size 1.27 1.27)) (justify left bottom))
   )
@@
     )
   )
+  (global_label "+5V_PICO" (shape input) (at 259.08 226.06 0) (fields_autoplaced)
+    (effects (font (size 1.27 1.27)) (justify left))
+    (property "Intersheetrefs" "${INTERSHEET_REFS}" (at 271.3786 226.06 0)
+      (effects (font (size 1.27 1.27)) (justify left) hide)
+    )
+  )
   (global_label "+3V3_ISO" (shape input) (at 181.61 284.48 180) (fields_autoplaced)
     (effects (font (size 1.27 1.27)) (justify right))
@@
     )
   )
-  (global_label "+3V3_ISO" (shape input) (at 248.92 276.86 0) (fields_autoplaced)
+  (global_label "+5V_PICO" (shape input) (at 248.92 276.86 0) (fields_autoplaced)
     (effects (font (size 1.27 1.27)) (justify left))
-    (property "Intersheetrefs" "${INTERSHEET_REFS}" (at 261.0976 276.86 0)
+    (property "Intersheetrefs" "${INTERSHEET_REFS}" (at 261.2186 276.86 0)
       (effects (font (size 1.27 1.27)) (justify left) hide)
     )
@@
     )
   )
+  (symbol (lib_id "power:GNDA") (at 259.08 229.87 0) (unit 1)
+    (in_bom yes) (on_board yes) (dnp no) (fields_autoplaced)
+    (property "Reference" "#PWR064" (at 259.08 236.22 0)
+      (effects (font (size 1.27 1.27)) hide)
+    )
+    (property "Value" "GNDA" (at 259.08 234.95 0)
+      (effects (font (size 1.27 1.27)))
+    )
+    (property "Footprint" "" (at 259.08 229.87 0)
+      (effects (font (size 1.27 1.27)) hide)
+    )
+    (property "Datasheet" "" (at 259.08 229.87 0)
+      (effects (font (size 1.27 1.27)) hide)
+    )
+    (pin "1")
+    (instances
+      (project "energy_meter"
+        (path "/911e1b35-25a5-4acc-afe7-a5e849f2ebf2"
+          (reference "#PWR064") (unit 1)
+        )
+      )
+    )
+  )
   (symbol (lib_id "Device:R_US") (at 95.25 39.37 90) (unit 1)
     (in_bom yes) (on_board yes) (dnp no) (fields_autoplaced)
@@
         )
       )
+    )
+  )
+  (symbol (lib_id "Connector:Screw_Terminal_01x02") (at 251.46 228.6 180) (unit 1)
+    (in_bom yes) (on_board yes) (dnp no) (fields_autoplaced)
+    (property "Reference" "J8" (at 251.46 219.71 0)
+      (effects (font (size 1.27 1.27)))
+    )
+    (property "Value" "5V_SMPS" (at 251.46 222.25 0)
+      (effects (font (size 1.27 1.27)))
+    )
+    (property "Footprint" "" (at 251.46 228.6 0)
+      (effects (font (size 1.27 1.27)) hide)
+    )
+    (property "Datasheet" "~" (at 251.46 228.6 0)
+      (effects (font (size 1.27 1.27)) hide)
+    )
+    (pin "2")
+    (pin "1")
+    (instances
+      (project "energy_meter"
+        (path "/911e1b35-25a5-4acc-afe7-a5e849f2ebf2"
+          (reference "J8") (unit 1)
+        )
+      )

Commit message: finish schematic started on layout
Parts:
- added BZ1: Buzzer, Buzzer_Beeper:Buzzer_12x9.5RM7.6, symbol Device:Buzzer
- added C49: 0.1u, Capacitor_SMD:C_0805_2012Metric_Pad1.18x1.45mm_HandSolder, symbol Device:C
- added C50: 22u, Capacitor_SMD:C_0805_2012Metric_Pad1.18x1.45mm_HandSolder, symbol Device:C
- added J10: EARTH, TerminalBlock_Phoenix:TerminalBlock_Phoenix_MKDS-1,5-2_1x02_P5.00mm_Horizontal, symbol Connector:Screw_Terminal_01x02
- added J9: IA_in, TerminalBlock_Phoenix:TerminalBlock_Phoenix_MKDS-1,5-2_1x02_P5.00mm_Horizontal, symbol Connector:Screw_Terminal_01x02
- added Q1: Q_NMOS_SGD, Package_TO_SOT_SMD:SOT-23, symbol Device:Q_NMOS_GSD
- added R34: 10k, Resistor_SMD:R_0805_2012Metric_Pad1.20x1.40mm_HandSolder, symbol Device:R_US
- added R35: 1k, Resistor_SMD:R_0805_2012Metric_Pad1.20x1.40mm_HandSolder, symbol Device:R_US
- added U5: BME280, BME280_beakout:BME_breakout, symbol BME280_breakout:BME280_breakout
- added U6: AMS1117-3.3, Package_TO_SOT_SMD:SOT-223-3_TabPin2, symbol Regulator_Linear:AMS1117-3.3
- C21: value 4.7u -> 10u
- J5, J6, J7: symbol Connector_Generic_MountingPin:Conn_01x01_MountingPin -> Connector_Generic:Conn_01x01
- J8: footprint (none) -> TerminalBlock_Phoenix:TerminalBlock_Phoenix_MKDS-1,5-2_1x02_P5.00mm_Horizontal
- T1: value T60404-E4626-X502 -> IA_in
- T2: value T60404-E4626-X502 -> IB_in
Connections:
- net +3V3_ADE: now also C20.1, C21.1, U1.1 (PULL_HIGH)
- net +3V3_ISO: now also U5.1 (VCC), U6.2 (VO); no longer C20.1, C21.1, U1.1 (PULL_HIGH)
- net +5V_PICO: now also BZ1.1 (+), C49.1, C50.1, U6.3 (VI)
- net GNDA: now also C49.2, C50.2, Q1.2 (S), R34.2, U5.2 (GND), U5.6 (SDO), U6.1 (GND)
- net SCL_PICO: now also U5.3 (SCL)
- net SDA_PICO: now also U5.4 (SDA)
- net at CR1.2, CR2.1, R13.1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: now also J9.2 (Pin_2)
- net at CR1.1, CR2.2, R11.1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: now also J9.1 (Pin_1)
- net BUZZER: now reaches U4.20 (GPIO15)
- net BUZZER: now also Q1.1 (G), R34.1
- net at CR3.1, CR4.2, R17.1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: now also J10.1 (Pin_1)
- net at CR3.2, CR4.1, R18.2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: now also J10.2 (Pin_2)
- new net: Q1.3 (D), R35.2
- new net: BZ1.2 (-), R35.1
- no-connect marks 14 -> 33
Other:
- note removed: "Is this even needed if we don't need the level shift"
- note removed: "What? Why is 3V3_ISO here?"
- moved on the sheet: C10, C20, C21, C39, C40, C41, C42, C43, C44, C6, C7, C9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
