File: energy_meter/central.kicad_sch (KiCad schematic)
At the start: 0 parts

Commit message: Example code
Parts:
- added D9: D_Schottky, symbol Device:D_Schottky
- added J11: Conn_01x02, symbol Connector_Generic:Conn_01x02
- added U7: Pico_SMD_NODEBUG, RPi_Pico:RPi_Pico_SMD, symbol RPi Pico:Pico_SMD_NODEBUG
Connections:
- new net: D9.1 (K), U7.39 (VSYS)
- new net GND1: J11.1 (Pin_1)
- new net PWR_IN: D9.2 (A), J11.2 (Pin_2)
Changed lines of the file:
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@@
     (company "Group TUE-01, EE344 \\nAutodialing alarm system for temperature and humidity monitoring\\n\\n\\n\\n")
   )
+  (wire (pts (xy 166.37 69.85) (xy 172.72 69.85))
+    (stroke (width 0) (type default))
+  )
+  (wire (pts (xy 88.9 72.39) (xy 88.9 74.93))
+    (stroke (width 0) (type default))
+  )
+  (wire (pts (xy 180.34 69.85) (xy 186.69 69.85))
+    (stroke (width 0) (type default))
+  )
+  (wire (pts (xy 86.36 69.85) (xy 91.44 69.85))
+    (stroke (width 0) (type default))
+  )
+  (wire (pts (xy 86.36 72.39) (xy 88.9 72.39))
+    (stroke (width 0) (type default))
+  )
+  (global_label "PWR_IN" (shape input) (at 186.69 69.85 0) (fields_autoplaced)
+    (effects (font (size 1.27 1.27)) (justify left))
+    (property "Intersheetrefs" "${INTERSHEET_REFS}" (at 196.5695 69.85 0)
+      (effects (font (size 1.27 1.27)) (justify left) hide)
+    )
+  )
+  (global_label "PWR_IN" (shape input) (at 91.44 69.85 0) (fields_autoplaced)
+    (effects (font (size 1.27 1.27)) (justify left))
+    (property "Intersheetrefs" "${INTERSHEET_REFS}" (at 101.3195 69.85 0)
+      (effects (font (size 1.27 1.27)) (justify left) hide)
+    )
+  )
+  (symbol (lib_id "power:GND1") (at 88.9 74.93 0) (unit 1)
+    (in_bom yes) (on_board yes) (dnp no) (fields_autoplaced)
+    (property "Reference" "#PWR069" (at 88.9 81.28 0)
+      (effects (font (size 1.27 1.27)) hide)
+    )
+    (property "Value" "GND1" (at 88.9 80.01 0)
+      (effects (font (size 1.27 1.27)))
+    )
+    (property "Footprint" "" (at 88.9 74.93 0)
+      (effects (font (size 1.27 1.27)) hide)
+    )
+    (property "Datasheet" "" (at 88.9 74.93 0)
+      (effects (font (size 1.27 1.27)) hide)
+    )
+    (pin "1")
+    (instances
+      (project "energy_meter"
+        (path "/911e1b35-25a5-4acc-afe7-a5e849f2ebf2/d6ad050f-ccf3-4675-8ea4-c04e775147fe"
+          (reference "#PWR069") (unit 1)
+        )
+      )
+    )
+  )
+  (symbol (lib_id "Connector_Generic:Conn_01x02") (at 81.28 72.39 180) (unit 1)
+    (in_bom yes) (on_board yes) (dnp no) (fields_autoplaced)
+    (property "Reference" "J11" (at 81.28 63.5 0)
+      (effects (font (size 1.27 1.27)))
+    )
+    (property "Value" "Conn_01x02" (at 81.28 66.04 0)
+      (effects (font (size 1.27 1.27)))
+    )
+    (property "Footprint" "" (at 81.28 72.39 0)
+      (effects (font (size 1.27 1.27)) hide)
+    )
+    (property "Datasheet" "~" (at 81.28 72.39 0)
+      (effects (font (size 1.27 1.27)) hide)
+    )
+    (pin "2")
+    (pin "1")
+    (instances
+      (project "energy_meter"
+        (path "/911e1b35-25a5-4acc-afe7-a5e849f2ebf2/d6ad050f-ccf3-4675-8ea4-c04e775147fe"
+          (reference "J11") (unit 1)
+        )
+      )
+    )
+  )
+  (symbol (lib_id "Device:D_Schottky") (at 176.53 69.85 0) (unit 1)
+    (in_bom yes) (on_board yes) (dnp no) (fields_autoplaced)
+    (property "Reference" "D9" (at 176.2125 63.5 0)
+      (effects (font (size 1.27 1.27)))
+    )
+    (property "Value" "D_Schottky" (at 176.2125 66.04 0)
+      (effects (font (size 1.27 1.27)))
+    )
+    (property "Footprint" "" (at 176.53 69.85 0)
+      (effects (font (size 1.27 1.27)) hide)
+    )
+    (property "Datasheet" "~" (at 176.53 69.85 0)
+      (effects (font (size 1.27 1.27)) hide)
+    )
+    (pin "1")
+    (pin "2")
+    (instances
+      (project "energy_meter"
+        (path "/911e1b35-25a5-4acc-afe7-a5e849f2ebf2/d6ad050f-ccf3-4675-8ea4-c04e775147fe"
+          (reference "D9") (unit 1)
+        )
+      )
+    )
+  )
+  (symbol (lib_id "RPi Pico:Pico_SMD_NODEBUG") (at 148.59 91.44 0) (unit 1)
+    (in_bom yes) (on_board yes) (dnp no) (fields_autoplaced)
+    (property "Reference" "U7" (at 148.59 59.69 0)
+      (effects (font (size 1.27 1.27)))
+    )
+    (property "Value" "Pico_SMD_NODEBUG" (at 148.59 62.23 0)
+      (effects (font (size 1.27 1.27)))
+    )
+    (property "Footprint" "RPi_Pico:RPi_Pico_SMD" (at 148.59 91.44 90)
+      (effects (font (size 1.27 1.27)) hide)
+    )
+    (property "Datasheet" "" (at 148.59 91.44 0)
+      (effects (font (size 1.27 1.27)) hide)
+    )
+    (pin "9")
+    (pin "35")
+    (pin "5")
+    (pin "18")
+    (pin "27")
+    (pin "34")
+    (pin "32")
+    (pin "16")
+    (pin "36")
+    (pin "31")
+    (pin "14")
+    (pin "7")
+    (pin "39")
+    (pin "33")
+    (pin "26")
+    (pin "38")
+    (pin "12")
+    (pin "11")
+    (pin "2")
+    (pin "24")
+    (pin "8")
+    (pin "37")
+    (pin "30")
+    (pin "21")
+    (pin "23")
+    (pin "25")
+    (pin "4")
+    (pin "40")
+    (pin "29")
+    (pin "28")
+    (pin "22")
+    (pin "19")
+    (pin "3")
+    (pin "15")
+    (pin "17")
+    (pin "13")
+    (pin "20")
+    (pin "1")
+    (pin "6")
+    (pin "10")
+    (instances
+      (project "energy_meter"
+        (path "/911e1b35-25a5-4acc-afe7-a5e849f2ebf2/d6ad050f-ccf3-4675-8ea4-c04e775147fe"
+          (reference "U7") (unit 1)
+        )
+      )
+    )
+  )
 )
