File: energy_meter/energy_meter.kicad_pcb (KiCad board)
At the start: 2 copper layers, 120 x 115 mm, 157 parts, among them IC1 ADUM4151BRIZ, IC2 ADUM6404ARIZ, IC3 ADP122AUJZ-3.3-R7, IC4 24LC32A_SN, J1 Screw_Terminal_01x02, J10 IB_in, J2 Screw_Terminal_01x02, J3 MicroUSB, J8 5V_SMPS, J9 IA_in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

Commit message: finished layout
Parts:
- removed TP18, TP2, TP20, TP22, TP24, TP4, TP6, TP8: TestPoint, TestPoint:TestPoint_Pad_D1.5mm
- moved C31 250.8 mm to (109.6, 95.0)
- moved U3 250.3 mm to (102.9, 94.4), turned to 0 degrees
- moved C28 239.9 mm to (94.4, 100.6)
- moved C23 239.6 mm to (94.2, 83.8), turned to 180 degrees
- moved C29 236.7 mm to (94.4, 97.6)
- moved C30 235.6 mm to (94.4, 91.0), turned to 180 degrees
- moved C36 229.3 mm to (123.2, 94.6), turned to 180 degrees
- moved SW1 229.1 mm to (118.0, 81.2)
- moved R30 228.8 mm to (123.2, 91.4), turned to 180 degrees
- moved C24 228.6 mm to (81.4, 104.2), turned to -90 degrees
- moved D7 226.2 mm to (115.4, 95.2), turned to 90 degrees
- moved D6 226.1 mm to (115.4, 90.0), turned to -90 degrees
- moved C25 225.3 mm to (78.4, 104.2), turned to -90 degrees
- moved C13 225.1 mm to (70.3, 91.3), turned to -90 degrees
- moved C12 224.0 mm to (69.5, 80.3)
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
Commit message: more libraries
Parts:
- U1: footprint ade9000:ADE9000ACPZ_ADI-M -> ADE9000:ADE9000ACPZ_ADI
- U2, U3: footprint SN74LV4T125PWR:PW0014A_N -> SN74LV:PW0014A_N
- U4: footprint RPi Pico:RPi_PicoW_SMD -> RPi_Pico:RPi_PicoW_SMD
- moved R33 35.9 mm to (95.9, 66.8), turned to 90 degrees
- moved J3 1.39 mm to (140.6, 93.1)
- moved J8 1.19 mm to (139.1, 83.7)
- moved U4 0.46 mm to (117.9, 52.0)
Connections:
- U4 pad 10: MOSI_ISO -> unconnected-(U4-GPIO7-Pad10)
- U4 pad 11: MISO_ISO -> unconnected-(U4-GPIO8-Pad11)
- U4 pad 12: SS_ISO -> WS_LED
- U4 pad 21: unconnected-(U4-GPIO16-Pad21) -> MISO_ISO
- U4 pad 22: unconnected-(U4-GPIO17-Pad22) -> SS_ISO
- U4 pad 24: unconnected-(U4-GPIO18-Pad24) -> SCLK_ISO
- U4 pad 25: unconnected-(U4-GPIO19-Pad25) -> MOSI_ISO
- U4 pad 26: unconnected-(U4-GPIO20-Pad26) -> RESET_ISO
- U4 pad 27: WS_LED -> unconnected-(U4-GPIO21-Pad27)
- U4 pad 9: SCLK_ISO -> unconnected-(U4-GPIO6-Pad9)

Commit message: pcb routing1
Parts:
- removed TP1, TP10, TP11, TP12, TP13, TP14, TP15, TP16, TP17, TP19, TP21, TP23, TP25, TP26, TP27, TP28, TP29, TP3, TP30, TP31, TP32, TP5, TP7, TP9: TestPoint, TestPoint:TestPoint_Pad_D1.5mm
- moved T2 30.5 mm to (38.4, 64.0), turned to -90 degrees
- moved R9 13.0 mm to (43.4, 116.2), turned to 90 degrees
- moved C4 12.6 mm to (57.4, 114.8), turned to 90 degrees
- moved C5 9.71 mm to (61.7, 118.4), turned to 0 degrees
- moved R15 8.05 mm to (60.2, 114.8), turned to -90 degrees
- moved R6 8.04 mm to (61.7, 106.2), turned to -90 degrees
- moved R3 6.37 mm to (51.6, 105.3), turned to -90 degrees
- moved R29 5.03 mm to (94.7, 71.4)
- moved C23 4.61 mm to (93.5, 79.2)
- moved C8 4.18 mm to (63.5, 114.8), turned to 90 degrees
- moved C2 3.43 mm to (60.2, 109.7), turned to 0 degrees
- moved FB1 3.24 mm to (38.9, 107.7)
- moved R2 2.90 mm to (47.5, 105.2), turned to 90 degrees
- moved C37 2.73 mm to (110.5, 79.5)
- moved C38 2.73 mm to (110.5, 83.3)
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Routing:
- net +3V3_ADE: track 0.00 -> 136.0 mm, vias 0 -> 4
- net BUZZER: track 0.00 -> 122.2 mm, vias 0 -> 2
- net IRQ0_ADE: track 0.00 -> 120.3 mm, vias 0 -> 4
- net DREADY_ADE: track 0.00 -> 110.7 mm, vias 0 -> 3
- net +3V3_ISO: track 0.00 -> 103.9 mm, vias 0 -> 4
- net +5V_PICO: track 0.00 -> 88.9 mm
- net IRQ1_ISO: track 0.00 -> 86.3 mm, vias 0 -> 2
- net SDA_PICO: track 0.00 -> 83.3 mm, vias 0 -> 2
- net ZX_ADE: track 0.00 -> 72.7 mm, vias 0 -> 2
- net RESET_ISO: track 0.00 -> 71.7 mm, vias 0 -> 2
- net SCL_PICO: track 0.00 -> 69.1 mm, vias 0 -> 2
- net RESET_ADE: track 0.00 -> 67.3 mm, vias 0 -> 2
- net IAP: track 0.00 -> 62.6 mm, vias 0 -> 2
- net PM1_ADE: track 0.00 -> 61.2 mm, vias 0 -> 3
- net ZX_ISO: track 0.00 -> 60.1 mm, vias 0 -> 2
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- added copper zone on B.Cu, net GND
- added copper zone on F.Cu, net GND
- added copper zone on B.Cu, net GNDA
- added copper zone on F.Cu, net GNDA
